Commit message: separate point and orientation match tasks. Breaks sensitivity for now

File: test/urdf/simple_atlas.urdf (robot description, URDF)
Before this commit: robot BoxAtlas, 13 links, 12 joints
Links:
- removed link floor
- removed link wall
- link l_foot_sole: mass 7.05 -> 0.2
- link l_foot_sole_dummy: mass 9.1 -> 0.0
- link l_hand_mount: mass 7.06 -> 0.05
- link l_hand_mount_dummy: mass 8.285 -> 0.0
- link pelvis: mass 112.12 -> 1.0
- link r_foot_sole: mass 7.05 -> 0.2
- link r_foot_sole_dummy: mass 9.1 -> 0.0
- link r_hand_mount: mass 7.06 -> 0.05
- link r_hand_mount_dummy: mass 8.285 -> 0.0
Joints:
- removed joint floor_to_wall
- removed joint root_to_floor
- joint pelvis_to_l_foot_sole_extension: limit lower=0.475 upper=0.95 effort=3000 velocity=100 -> lower=0.475 upper=0.95 effort=20 velocity=100
- joint pelvis_to_l_foot_sole_rotation: limit lower=-0.05 upper=0.785398 effort=530 velocity=100 -> lower=-0.05 upper=0.785398 effort=10 velocity=100
- joint pelvis_to_l_hand_mount_extension: axis 0 1 0 -> 0 0 1; limit lower=0.4 upper=0.8 effort=500 velocity=100 -> lower=0.4 upper=0.8 effort=2 velocity=100; origin xyz=0 0 0 rpy=1.5707963267948966 0 -1.5707963267948966 -> xyz=0 0 0
- joint pelvis_to_l_hand_mount_rotation: limit lower=0 upper=1.6708 effort=100 velocity=100 -> lower=0 upper=1.6708 effort=2 velocity=100
- joint pelvis_to_r_foot_sole_extension: limit lower=0.475 upper=0.95 effort=3000 velocity=100 -> lower=0.475 upper=0.95 effort=20 velocity=100
- joint pelvis_to_r_foot_sole_rotation: limit lower=-0.05 upper=0.785398 effort=530 velocity=100 -> lower=-0.05 upper=0.785398 effort=10 velocity=100
- joint pelvis_to_r_hand_mount_extension: axis 0 1 0 -> 0 0 1; limit lower=0.4 upper=0.8 effort=500 velocity=100 -> lower=0.4 upper=0.8 effort=2 velocity=100; origin xyz=0 0 0 rpy=1.5707963267948966 0 1.5707963267948966 -> xyz=0 0 0
- joint pelvis_to_r_hand_mount_rotation: limit lower=0 upper=1.6708 effort=100 velocity=100 -> lower=0 upper=1.6708 effort=2 velocity=100
